Commit message: Updated collector_controller_node.py

File: src/simulation_system/urdf/mycobot_280.urdf (robot description, URDF)
Before this commit: robot mycobot_280, 11 links, 9 joints
Joints:
- added joint collector_base_joint: type fixed, parent base_link, child collector_base, origin xyz=0.15 0 0.02 rpy=0 0 0
